Commit message: added lidar

File: autonomous_vehicle/src/my_robot_description/urdf/robot.urdf.xacro (robot description, xacro)
@@ -11,4 +11,5 @@
     <xacro:property name="wheel_thickness" value="0.04"/>
     <xacro:property name="wheel_separation" value="0.35"/>
+    <xacro:property name="base_height" value="${chassis_height}"/>
     <!-- Base Link (Chassis) -->
     <link name="base_link">
@@ -93,4 +94,49 @@
         </inertial>
     </link>
+    <link name="laser_frame">
+    <visual>
+      <geometry>
+        <cylinder length="0.03" radius="0.03"/>
+      </geometry>
+      <material name="red">
+        <color rgba="0.8 0.0 0.0 1.0"/>
+      </material>
+    </visual>
+  </link>
+  <joint name="laser_joint" type="fixed">
+    <parent link="base_link"/>
+    <child link="laser_frame"/>
+    <origin xyz="0 0 ${base_height/2 + 0.05}"/>
+  </joint>
+  <gazebo reference="laser_frame">
+    <sensor name="laser" type="ray">
+      <always_on>true</always_on>
+      <visualize>true</visualize>
+      <update_rate>10.0</update_rate>
+      <ray>
+        <scan>
+          <horizontal>
+            <samples>360</samples>
+            <resolution>1</resolution>
+            <min_angle>-3.14</min_angle>
+            <max_angle>3.14</max_angle>
+          </horizontal>
+        </scan>
+        <range>
+          <min>0.1</min>
+          <max>5.0</max>
+          <resolution>0.01</resolution>
+        </range>
+      </ray>
+      <plugin name="gazebo_ros_lidar_controller" filename="libgazebo_ros_ray_sensor.so">
+        <ros>
+          <argument>~/out:=scan</argument>
+          <remapping>~/out:=/scan</remapping>
+        </ros>
+        <output_type>sensor_msgs/LaserScan</output_type>
+        <frame_name>laser_frame</frame_name>
+      </plugin>
+    </sensor>
+  </gazebo>
     <!-- Joints -->
     <joint name="right_wheel_joint" type="continuous">
